File: pcb/revxlp.kicad_sch (KiCad schematic)
At the start: 134 parts, among them Q1 AO3416 N-channel MOSFET, SW1 SW_SPDT, SW2 SW_Push, U1 74HC595, U2 SeeeduinoXIAO_BLE

Commit message: Fix bottom row missing via, some better copper fills.
Parts:
- added R_AltG2: (no value), symbol Device:R_Small_US
- added SwAltG2: (no value), symbol Switch:SW_Push_LED
- D_G5: value (none) -> D; footprint (none) -> Diode_SMD:D_1206_3216Metric_Pad1.42x1.75mm_HandSolder
- Q1: LCSC Part Number (none) -> C479060
- R80: LCSC Part Number (none) -> C17936
- R_G5: value (none) -> R; footprint (none) -> Resistor_SMD:R_1206_3216Metric_Pad1.30x1.75mm_HandSolder
- SwG5: value (none) -> SW_Push; footprint (none) -> revxlp:PG1350_socket_smdLed
- U1: LCSC Part Number (none) -> C10092
Connections:
- net +5V: now also SwAltG2.4 (A)
- net col2: now also SwAltG2.2
- net ledOut: now also R_AltG2.1
- net at D_G2.2 (A), SwG2.1: now also SwAltG2.1
- new net: R_AltG2.2, SwAltG2.3 (K)
Changed lines of the file:
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@@
   (junction (at 175.26 78.74) (diameter 0) (color 0 0 0 0)
   )
+  (junction (at 102.87 160.02) (diameter 0) (color 0 0 0 0)
+  )
   (junction (at 34.29 171.45) (diameter 0) (color 0 0 0 0)
   )
@@
   (junction (at 85.09 69.85) (diameter 0) (color 0 0 0 0)
   )
+  (junction (at 105.41 162.56) (diameter 0) (color 0 0 0 0)
+  )
   (junction (at 54.61 60.96) (diameter 0) (color 0 0 0 0)
   )
@@
   (junction (at 85.09 171.45) (diameter 0) (color 0 0 0 0)
   )
+  (junction (at 89.535 160.02) (diameter 0) (color 0 0 0 0)
+  )
   (no_connect (at 217.17 103.505))
   (no_connect (at 261.62 154.94))
@@
     (stroke (width 0) (type default) (color 0 0 0 0))
   )
+  (wire (pts (xy 105.41 175.26) (xy 111.125 175.26))
+    (stroke (width 0) (type default) (color 0 0 0 0))
+  )
   (wire (pts (xy 40.64 78.74) (xy 34.29 78.74))
     (stroke (width 0) (type default) (color 0 0 0 0))
@@
     (stroke (width 0) (type default) (color 0 0 0 0))
   )
+  (wire (pts (xy 89.535 160.02) (xy 85.09 160.02))
+    (stroke (width 0) (type default) (color 0 0 0 0))
+  )
   (wire (pts (xy 57.15 133.35) (xy 57.15 153.67))
     (stroke (width 0) (type default) (color 0 0 0 0))
@@
     (stroke (width 0) (type default) (color 0 0 0 0))
   )
+  (wire (pts (xy 91.44 192.405) (xy 99.695 192.405))
+    (stroke (width 0) (type default) (color 0 0 0 0))
+  )
   (wire (pts (xy 175.26 78.74) (xy 175.26 99.06))
     (stroke (width 0) (type default) (color 0 0 0 0))
@@
     (stroke (width 0) (type default) (color 0 0 0 0))
   )
+  (wire (pts (xy 99.695 184.785) (xy 99.695 187.325))
+    (stroke (width 0) (type default) (color 0 0 0 0))
+  )
   (wire (pts (xy 139.7 72.39) (xy 115.57 72.39))
     (stroke (width 0) (type default) (color 0 0 0 0))
@@
     (stroke (width 0) (type default) (color 0 0 0 0))
   )
+  (wire (pts (xy 109.855 175.895) (xy 109.855 182.245))
+    (stroke (width 0) (type default) (color 0 0 0 0))
+  )
   (wire (pts (xy 115.57 113.03) (xy 91.44 113.03))
     (stroke (width 0) (type default) (color 0 0 0 0))
@@
     (stroke (width 0) (type default) (color 0 0 0 0))
   )
+  (wire (pts (xy 91.44 173.99) (xy 91.44 192.405))
+    (stroke (width 0) (type default) (color 0 0 0 0))
+  )
   (wire (pts (xy 81.28 101.6) (xy 81.28 121.92))
     (stroke (width 0) (type default) (color 0 0 0 0))
@@
     (stroke (width 0) (type default) (color 0 0 0 0))
   )
+  (wire (pts (xy 102.87 160.02) (xy 102.87 175.895))
+    (stroke (width 0) (type default) (color 0 0 0 0))
+  )
   (wire (pts (xy 102.87 78.74) (xy 101.6 78.74))
     (stroke (width 0) (type default) (color 0 0 0 0))
@@
     (stroke (width 0) (type default) (color 0 0 0 0))
   )
+  (wire (pts (xy 102.87 175.895) (xy 109.855 175.895))
+    (stroke (width 0) (type default) (color 0 0 0 0))
+  )
   (wire (pts (xy 67.31 160.02) (xy 60.96 160.02))
     (stroke (width 0) (type default) (color 0 0 0 0))
@@
     (stroke (width 0) (type default) (color 0 0 0 0))
   )
+  (wire (pts (xy 89.535 182.245) (xy 89.535 160.02))
+    (stroke (width 0) (type default) (color 0 0 0 0))
+  )
   (wire (pts (xy 57.15 153.67) (xy 57.15 173.99))
     (stroke (width 0) (type default) (color 0 0 0 0))
@@
     (stroke (width 0) (type default) (color 0 0 0 0))
   )
-  (wire (pts (xy 91.44 160.02) (xy 85.09 160.02))
+  (wire (pts (xy 91.44 160.02) (xy 89.535 160.02))
     (stroke (width 0) (type default) (color 0 0 0 0))
   )
@@
     (stroke (width 0) (type default) (color 0 0 0 0))
   )
+  (wire (pts (xy 111.125 175.26) (xy 111.125 184.785))
+    (stroke (width 0) (type default) (color 0 0 0 0))
+  )
   (wire (pts (xy 254 118.11) (xy 243.84 118.11))
     (stroke (width 0) (type default) (color 0 0 0 0))
@@
     (stroke (width 0) (type default) (color 0 0 0 0))
   )
+  (wire (pts (xy 111.125 184.785) (xy 109.855 184.785))
+    (stroke (width 0) (type default) (color 0 0 0 0))
+  )
   (wire (pts (xy 173.99 101.6) (xy 177.8 101.6))
     (stroke (width 0) (type default) (color 0 0 0 0))
@@
     (stroke (width 0) (type default) (color 0 0 0 0))
   )
+  (wire (pts (xy 105.41 162.56) (xy 105.41 175.26))
+    (stroke (width 0) (type default) (color 0 0 0 0))
+  )
   (wire (pts (xy 173.99 121.92) (xy 177.8 121.92))
     (stroke (width 0) (type default) (color 0 0 0 0))
@@
     (stroke (width 0) (type default) (color 0 0 0 0))
   )
+  (wire (pts (xy 99.695 182.245) (xy 89.535 182.245))
+    (stroke (width 0) (type default) (color 0 0 0 0))
+  )
   (wire (pts (xy 40.64 49.53) (xy 57.15 49.53))
     (stroke (width 0) (type default) (color 0 0 0 0))
@@
       (effects (font (size 1.27 1.27)) hide)
     )
+    (property "LCSC Part Number" "C17936" (id 4) (at 251.46 110.49 0)
+      (effects (font (size 1.27 1.27)) hide)
+    )
     (pin "1")
     (pin "2")
@@
       (effects (font (size 1.27 1.27)) hide)
     )
+    (property "LCSC Part Number" "C479060" (id 4) (at 259.08 115.57 90)
+      (effects (font (size 1.27 1.27)) hide)
+    )
     (pin "1")
     (pin "2")
@@
       (effects (font (size 1.27 1.27)) (justify right))
     )
-    (property "Value" "" (id 1) (at 165.5572 168.783 0)
+    (property "Value" "R" (id 1) (at 165.5572 168.783 0)
       (effects (font (size 1.27 1.27)) (justify right))
     )
-    (property "Footprint" "" (id 2) (at 163.83 167.64 0)
+    (property "Footprint" "Resistor_SMD:R_1206_3216Metric_Pad1.30x1.75mm_HandSolder" (id 2) (at 163.83 167.64 0)
       (effects (font (size 1.27 1.27)) hide)
     )
@@
     (in_bom yes) (on_board yes)
     (property "Reference" "SwG5" (id 0) (at 168.91 155.321 0))
-    (property "Value" "" (id 1) (at 168.91 157.6324 0))
-    (property "Footprint" "" (id 2) (at 168.91 157.48 0)
+    (property "Value" "SW_Push" (id 1) (at 168.91 157.6324 0))
+    (property "Footprint" "revxlp:PG1350_socket_smdLed" (id 2) (at 168.91 157.48 0)
       (effects (font (size 1.27 1.27)) hide)
     )
@@
       (effects (font (size 1.27 1.27)) hide)
     )
+    (property "LCSC Part Number" "C10092" (id 4) (at 207.01 111.125 0)
+      (effects (font (size 1.27 1.27)) hide)
+    )
     (pin "1")
     (pin "10")
@@
     (pin "1")
   )
+  (symbol (lib_id "Device:R_Small_US") (at 99.695 189.865 180) (unit 1)
+    (in_bom yes) (on_board yes)
+    (property "Reference" "R_AltG2" (id 0) (at 101.4222 188.6966 0)
+      (effects (font (size 1.27 1.27)) (justify right))
+    )
+    (property "Value" "" (id 1) (at 101.4222 191.008 0)
+      (effects (font (size 1.27 1.27)) (justify right))
+    )
+    (property "Footprint" "" (id 2) (at 99.695 189.865 0)
+      (effects (font (size 1.27 1.27)) hide)
+    )
+    (property "Datasheet" "~" (id 3) (at 99.695 189.865 0)
+      (effects (font (size 1.27 1.27)) hide)
+    )
+    (pin "1")
+    (pin "2")
+  )
+  (symbol (lib_id "Switch:SW_Push_LED") (at 104.775 184.785 0) (unit 1)
+    (in_bom yes) (on_board yes)
+    (property "Reference" "SwAltG2" (id 0) (at 104.775 177.546 0))
+    (property "Value" "" (id 1) (at 104.775 179.8574 0))
+    (property "Footprint" "" (id 2) (at 104.775 179.705 0)
+      (effects (font (size 1.27 1.27)) hide)
+    )
+    (property "Datasheet" "~" (id 3) (at 104.775 179.705 0)
+      (effects (font (size 1.27 1.27)) hide)
+    )
+    (pin "1")
+    (pin "2")
+    (pin "3")
+    (pin "4")
+  )
   (symbol (lib_id "Device:D") (at 157.48 163.83 90) (unit 1)
     (in_bom yes) (on_board yes)
@@
       (effects (font (size 1.27 1.27)) (justify right))
     )
-    (property "Value" "" (id 1) (at 159.512 164.973 90)
+    (property "Value" "D" (id 1) (at 159.512 164.973 90)
       (effects (font (size 1.27 1.27)) (justify right))
     )
-    (property "Footprint" "" (id 2) (at 157.48 163.83 0)
+    (property "Footprint" "Diode_SMD:D_1206_3216Metric_Pad1.42x1.75mm_HandSolder" (id 2) (at 157.48 163.83 0)
       (effects (font (size 1.27 1.27)) hide)
     )
@@
       (reference "R_A5") (unit 1) (value "R") (footprint "Resistor_SMD:R_1206_3216Metric_Pad1.30x1.75mm_HandSolder")
     )
+    (path "/dca9abab-49c2-4d6d-88f5-a24a9063e847"
+      (reference "R_AltG2") (unit 1) (value "R") (footprint "Resistor_SMD:R_1206_3216Metric_Pad1.30x1.75mm_HandSolder")
+    )
     (path "/00000000-0000-0000-0000-000060a89d01"
       (reference "R_B0") (unit 1) (value "R") (footprint "Resistor_SMD:R_1206_3216Metric_Pad1.30x1.75mm_HandSolder")
@@
       (reference "SwA5") (unit 1) (value "SW_Push") (footprint "revxlp:PG1350_socket_smdLed")
     )
+    (path "/ef914691-5491-42fb-853b-5015433cd48c"
+      (reference "SwAltG2") (unit 1) (value "SW_Push") (footprint "revxlp:PG1350_socket_smdLed")
+    )
     (path "/00000000-0000-0000-0000-000060a89cf5"

Commit message: Add JST socket, various tweaks/fixes.
Parts:
- added BT2: Battery_Cell, Connector_JST:JST_SH_SM02B-SRSS-TB_1x02-1MP_P1.00mm_Horizontal, symbol Device:Battery_Cell
- R_AltG2: value (none) -> R; footprint (none) -> Resistor_SMD:R_1206_3216Metric_Pad1.30x1.75mm_HandSolder
- SwAltG2: value (none) -> SW_Push; footprint (none) -> revxlp:PG1350_socket_smdLed
Connections:
- net BAT+: now also BT2.2 (+)
- net at BT1.2 (-), SW1.1 (A): now also BT2.1 (-)
Changed lines of the file:
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@@
   (junction (at 102.87 35.56) (diameter 0) (color 0 0 0 0)
   )
+  (junction (at 264.795 149.86) (diameter 0) (color 0 0 0 0)
+  )
   (junction (at 57.15 173.99) (diameter 0) (color 0 0 0 0)
   )
@@
     (stroke (width 0) (type default) (color 0 0 0 0))
   )
+  (wire (pts (xy 264.795 149.86) (xy 264.795 161.29))
+    (stroke (width 0) (type default) (color 0 0 0 0))
+  )
   (wire (pts (xy 81.28 101.6) (xy 81.28 121.92))
     (stroke (width 0) (type default) (color 0 0 0 0))
@@
     (stroke (width 0) (type default) (color 0 0 0 0))
   )
+  (wire (pts (xy 264.795 161.29) (xy 266.7 161.29))
+    (stroke (width 0) (type default) (color 0 0 0 0))
+  )
   (wire (pts (xy 40.64 99.06) (xy 34.29 99.06))
     (stroke (width 0) (type default) (color 0 0 0 0))
@@
     (stroke (width 0) (type default) (color 0 0 0 0))
   )
+  (wire (pts (xy 264.795 149.86) (xy 266.7 149.86))
+    (stroke (width 0) (type default) (color 0 0 0 0))
+  )
   (wire (pts (xy 105.41 60.96) (xy 105.41 81.28))
     (stroke (width 0) (type default) (color 0 0 0 0))
@@
     (stroke (width 0) (type default) (color 0 0 0 0))
   )
+  (wire (pts (xy 274.32 161.29) (xy 277.495 161.29))
+    (stroke (width 0) (type default) (color 0 0 0 0))
+  )
   (wire (pts (xy 81.28 38.1) (xy 81.28 52.07))
     (stroke (width 0) (type default) (color 0 0 0 0))
@@
     (stroke (width 0) (type default) (color 0 0 0 0))
   )
-  (wire (pts (xy 261.62 149.86) (xy 266.7 149.86))
+  (wire (pts (xy 261.62 149.86) (xy 264.795 149.86))
     (stroke (width 0) (type default) (color 0 0 0 0))
   )
@@
     (stroke (width 0) (type default) (color 0 0 0 0))
   )
+  (wire (pts (xy 274.32 149.86) (xy 277.495 149.86))
+    (stroke (width 0) (type default) (color 0 0 0 0))
+  )
+  (wire (pts (xy 277.495 149.86) (xy 277.495 161.29))
+    (stroke (width 0) (type default) (color 0 0 0 0))
+  )
   (wire (pts (xy 85.09 69.85) (xy 60.96 69.85))
     (stroke (width 0) (type default) (color 0 0 0 0))
@@
     )
   )
-  (global_label "BAT+" (shape input) (at 274.32 149.86 0) (fields_autoplaced)
+  (global_label "BAT+" (shape input) (at 277.495 155.575 0) (fields_autoplaced)
     (effects (font (size 1.27 1.27)) (justify left))
-    (property "Intersheet References" "${INTERSHEET_REFS}" (id 0) (at 281.5428 149.7806 0)
+    (property "Intersheet References" "${INTERSHEET_REFS}" (id 0) (at 284.7178 155.4956 0)
       (effects (font (size 1.27 1.27)) (justify left) hide)
     )
@@
     (pin "1")
   )
+  (symbol (lib_name "Battery_Cell_1") (lib_id "Device:Battery_Cell") (at 269.24 161.29 270) (unit 1)
+    (in_bom yes) (on_board yes)
+    (property "Reference" "BT2" (id 0) (at 275.59 162.56 90))
+    (property "Value" "Battery_Cell" (id 1) (at 273.05 162.56 90))
+    (property "Footprint" "Connector_JST:JST_SH_SM02B-SRSS-TB_1x02-1MP_P1.00mm_Horizontal" (id 2) (at 269.24 162.814 90)
+      (effects (font (size 1.27 1.27)) hide)
+    )
+    (property "Datasheet" "~" (id 3) (at 269.24 162.814 90)
+      (effects (font (size 1.27 1.27)) hide)
+    )
+    (pin "1")
+    (pin "2")
+  )
   (symbol (lib_id "power:+3V3") (at 260.35 45.72 0) (unit 1)
     (in_bom yes) (on_board yes) (fields_autoplaced)
@@
       (effects (font (size 1.27 1.27)) (justify right))
     )
-    (property "Value" "" (id 1) (at 101.4222 191.008 0)
+    (property "Value" "R" (id 1) (at 101.4222 191.008 0)
       (effects (font (size 1.27 1.27)) (justify right))
     )
-    (property "Footprint" "" (id 2) (at 99.695 189.865 0)
+    (property "Footprint" "Resistor_SMD:R_1206_3216Metric_Pad1.30x1.75mm_HandSolder" (id 2) (at 99.695 189.865 0)
       (effects (font (size 1.27 1.27)) hide)
     )
@@
     (in_bom yes) (on_board yes)
     (property "Reference" "SwAltG2" (id 0) (at 104.775 177.546 0))
-    (property "Value" "" (id 1) (at 104.775 179.8574 0))
-    (property "Footprint" "" (id 2) (at 104.775 179.705 0)
+    (property "Value" "SW_Push" (id 1) (at 104.775 179.8574 0))
+    (property "Footprint" "revxlp:PG1350_socket_smdLed" (id 2) (at 104.775 179.705 0)
       (effects (font (size 1.27 1.27)) hide)
     )
@@
       (reference "BT1") (unit 1) (value "Battery_Cell") (footprint "revxlp:cell_pads")
     )
+    (path "/8ada82cf-69cd-4e4a-977d-e16b6f21e2f9"
+      (reference "BT2") (unit 1) (value "Battery_Cell") (footprint "Connector_JST:JST_SH_SM02B-SRSS-TB_1x02-1MP_P1.00mm_Horizontal")
+    )
     (path "/00000000-0000-0000-0000-0000604dd7fe"
