File: pcb/revxlp.kicad_sch (KiCad schematic)
At the start: 137 parts, among them Q1 AO3416 N-channel MOSFET, SW1 SW_SPDT, SW2 SW_Push, U1 74HC595, U2 SeeeduinoXIAO_BLE

Commit message: Add mounting holes for a bottom plate w/ solder nuts.
Parts:
- added H1, H2, H3, H4, H5, H6: MountingHole, MountingHole:MountingHole_3mm_Pad_TopOnly, symbol Mechanical:MountingHole
Changed lines of the file:
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@@
     (pin "9")
+  )
+  (symbol (lib_id "Mechanical:MountingHole") (at 221.615 151.765 0) (unit 1)
+    (in_bom yes) (on_board yes) (fields_autoplaced)
+    (property "Reference" "H2" (id 0) (at 224.155 150.9303 0)
+      (effects (font (size 1.27 1.27)) (justify left))
+    )
+    (property "Value" "MountingHole" (id 1) (at 224.155 153.4672 0)
+      (effects (font (size 1.27 1.27)) (justify left))
+    )
+    (property "Footprint" "MountingHole:MountingHole_3mm_Pad_TopOnly" (id 2) (at 221.615 151.765 0)
+      (effects (font (size 1.27 1.27)) hide)
+    )
+    (property "Datasheet" "~" (id 3) (at 221.615 151.765 0)
+      (effects (font (size 1.27 1.27)) hide)
+    )
+  )
+  (symbol (lib_id "Mechanical:MountingHole") (at 213.995 158.75 0) (unit 1)
+    (in_bom yes) (on_board yes) (fields_autoplaced)
+    (property "Reference" "H5" (id 0) (at 216.535 157.9153 0)
+      (effects (font (size 1.27 1.27)) (justify left))
+    )
+    (property "Value" "MountingHole" (id 1) (at 216.535 160.4522 0)
+      (effects (font (size 1.27 1.27)) (justify left))
+    )
+    (property "Footprint" "MountingHole:MountingHole_3mm_Pad_TopOnly" (id 2) (at 213.995 158.75 0)
+      (effects (font (size 1.27 1.27)) hide)
+    )
+    (property "Datasheet" "~" (id 3) (at 213.995 158.75 0)
+      (effects (font (size 1.27 1.27)) hide)
+    )
   )
   (symbol (lib_id "Seeeduino XIAO:SeeeduinoXIAO_BLE") (at 227.33 49.53 0) (unit 1)
@@
     (pin "1")
   )
+  (symbol (lib_id "Mechanical:MountingHole") (at 231.14 161.925 0) (unit 1)
+    (in_bom yes) (on_board yes) (fields_autoplaced)
+    (property "Reference" "H6" (id 0) (at 233.68 161.0903 0)
+      (effects (font (size 1.27 1.27)) (justify left))
+    )
+    (property "Value" "MountingHole" (id 1) (at 233.68 163.6272 0)
+      (effects (font (size 1.27 1.27)) (justify left))
+    )
+    (property "Footprint" "MountingHole:MountingHole_3mm_Pad_TopOnly" (id 2) (at 231.14 161.925 0)
+      (effects (font (size 1.27 1.27)) hide)
+    )
+    (property "Datasheet" "~" (id 3) (at 231.14 161.925 0)
+      (effects (font (size 1.27 1.27)) hide)
+    )
+  )
   (symbol (lib_name "Battery_Cell_1") (lib_id "Device:Battery_Cell") (at 269.24 161.29 270) (unit 1)
     (in_bom yes) (on_board yes)
@@
     (pin "1")
   )
+  (symbol (lib_id "Mechanical:MountingHole") (at 182.245 161.925 0) (unit 1)
+    (in_bom yes) (on_board yes) (fields_autoplaced)
+    (property "Reference" "H3" (id 0) (at 184.785 161.0903 0)
+      (effects (font (size 1.27 1.27)) (justify left))
+    )
+    (property "Value" "MountingHole" (id 1) (at 184.785 163.6272 0)
+      (effects (font (size 1.27 1.27)) (justify left))
+    )
+    (property "Footprint" "MountingHole:MountingHole_3mm_Pad_TopOnly" (id 2) (at 182.245 161.925 0)
+      (effects (font (size 1.27 1.27)) hide)
+    )
+    (property "Datasheet" "~" (id 3) (at 182.245 161.925 0)
+      (effects (font (size 1.27 1.27)) hide)
+    )
+  )
+  (symbol (lib_id "Mechanical:MountingHole") (at 183.515 152.4 0) (unit 1)
+    (in_bom yes) (on_board yes) (fields_autoplaced)
+    (property "Reference" "H1" (id 0) (at 186.055 151.5653 0)
+      (effects (font (size 1.27 1.27)) (justify left))
+    )
+    (property "Value" "MountingHole" (id 1) (at 186.055 154.1022 0)
+      (effects (font (size 1.27 1.27)) (justify left))
+    )
+    (property "Footprint" "MountingHole:MountingHole_3mm_Pad_TopOnly" (id 2) (at 183.515 152.4 0)
+      (effects (font (size 1.27 1.27)) hide)
+    )
+    (property "Datasheet" "~" (id 3) (at 183.515 152.4 0)
+      (effects (font (size 1.27 1.27)) hide)
+    )
+  )
   (symbol (lib_id "Device:R_Small_US") (at 99.695 189.865 180) (unit 1)
     (in_bom yes) (on_board yes)
@@
     (pin "1")
     (pin "2")
+  )
+  (symbol (lib_id "Mechanical:MountingHole") (at 190.5 158.75 0) (unit 1)
+    (in_bom yes) (on_board yes) (fields_autoplaced)
+    (property "Reference" "H4" (id 0) (at 193.04 157.9153 0)
+      (effects (font (size 1.27 1.27)) (justify left))
+    )
+    (property "Value" "MountingHole" (id 1) (at 193.04 160.4522 0)
+      (effects (font (size 1.27 1.27)) (justify left))
+    )
+    (property "Footprint" "MountingHole:MountingHole_3mm_Pad_TopOnly" (id 2) (at 190.5 158.75 0)
+      (effects (font (size 1.27 1.27)) hide)
+    )
+    (property "Datasheet" "~" (id 3) (at 190.5 158.75 0)
+      (effects (font (size 1.27 1.27)) hide)
+    )
   )
   (symbol (lib_id "Switch:SW_Push_LED") (at 104.775 184.785 0) (unit 1)
@@
       (reference "D_G5") (unit 1) (value "D") (footprint "Diode_SMD:D_1206_3216Metric_Pad1.42x1.75mm_HandSolder")
     )
+    (path "/d668e699-ab17-4569-8fb7-e32e8aaed59e"
+      (reference "H1") (unit 1) (value "MountingHole") (footprint "MountingHole:MountingHole_3mm_Pad_TopOnly")
+    )
+    (path "/50f54e4b-0933-4757-9ac9-2f865ea8908e"
+      (reference "H2") (unit 1) (value "MountingHole") (footprint "MountingHole:MountingHole_3mm_Pad_TopOnly")
+    )
+    (path "/be5350c1-fa86-43a9-b1d8-e189608ad5ac"
+      (reference "H3") (unit 1) (value "MountingHole") (footprint "MountingHole:MountingHole_3mm_Pad_TopOnly")
+    )
+    (path "/e89d20fd-de0f-4c68-89c7-445e7cb108d7"
+      (reference "H4") (unit 1) (value "MountingHole") (footprint "MountingHole:MountingHole_3mm_Pad_TopOnly")
+    )
+    (path "/62f0725c-6ab8-4cb9-bc3d-061d4f32a171"
+      (reference "H5") (unit 1) (value "MountingHole") (footprint "MountingHole:MountingHole_3mm_Pad_TopOnly")
+    )
+    (path "/87ebb9fd-6588-4af4-b1d3-9119acfaa6a6"
+      (reference "H6") (unit 1) (value "MountingHole") (footprint "MountingHole:MountingHole_3mm_Pad_TopOnly")
+    )
     (path "/00000000-0000-0000-0000-00006075d32d"

Commit message: Add mounting holes, varios refactors.
Parts:
- added H7: MountingHole, revxlp:MountingHole_3mm_Pad_NonPTH_TopOnly, symbol Mechanical:MountingHole
- H1, H2, H3, H4, H5, H6: footprint MountingHole:MountingHole_3mm_Pad_TopOnly -> revxlp:MountingHole_3mm_Pad_NonPTH_TopOnly
Changed lines of the file:
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@@
       (effects (font (size 1.27 1.27)) (justify left))
     )
-    (property "Footprint" "MountingHole:MountingHole_3mm_Pad_TopOnly" (id 2) (at 221.615 151.765 0)
+    (property "Footprint" "revxlp:MountingHole_3mm_Pad_NonPTH_TopOnly" (id 2) (at 221.615 151.765 0)
       (effects (font (size 1.27 1.27)) hide)
     )
@@
       (effects (font (size 1.27 1.27)) (justify left))
     )
-    (property "Footprint" "MountingHole:MountingHole_3mm_Pad_TopOnly" (id 2) (at 213.995 158.75 0)
+    (property "Footprint" "revxlp:MountingHole_3mm_Pad_NonPTH_TopOnly" (id 2) (at 213.995 158.75 0)
       (effects (font (size 1.27 1.27)) hide)
     )
@@
     (pin "9")
   )
+  (symbol (lib_id "Mechanical:MountingHole") (at 203.2 151.13 0) (unit 1)
+    (in_bom yes) (on_board yes) (fields_autoplaced)
+    (property "Reference" "H7" (id 0) (at 205.74 150.2953 0)
+      (effects (font (size 1.27 1.27)) (justify left))
+    )
+    (property "Value" "MountingHole" (id 1) (at 205.74 152.8322 0)
+      (effects (font (size 1.27 1.27)) (justify left))
+    )
+    (property "Footprint" "revxlp:MountingHole_3mm_Pad_NonPTH_TopOnly" (id 2) (at 203.2 151.13 0)
+      (effects (font (size 1.27 1.27)) hide)
+    )
+    (property "Datasheet" "~" (id 3) (at 203.2 151.13 0)
+      (effects (font (size 1.27 1.27)) hide)
+    )
+  )
   (symbol (lib_id "power:+3V3") (at 207.01 95.885 0) (unit 1)
     (in_bom yes) (on_board yes) (fields_autoplaced)
@@
       (effects (font (size 1.27 1.27)) (justify left))
     )
-    (property "Footprint" "MountingHole:MountingHole_3mm_Pad_TopOnly" (id 2) (at 231.14 161.925 0)
+    (property "Footprint" "revxlp:MountingHole_3mm_Pad_NonPTH_TopOnly" (id 2) (at 231.14 161.925 0)
       (effects (font (size 1.27 1.27)) hide)
     )
@@
       (effects (font (size 1.27 1.27)) (justify left))
     )
-    (property "Footprint" "MountingHole:MountingHole_3mm_Pad_TopOnly" (id 2) (at 182.245 161.925 0)
+    (property "Footprint" "revxlp:MountingHole_3mm_Pad_NonPTH_TopOnly" (id 2) (at 182.245 161.925 0)
       (effects (font (size 1.27 1.27)) hide)
     )
@@
       (effects (font (size 1.27 1.27)) (justify left))
     )
-    (property "Footprint" "MountingHole:MountingHole_3mm_Pad_TopOnly" (id 2) (at 183.515 152.4 0)
+    (property "Footprint" "revxlp:MountingHole_3mm_Pad_NonPTH_TopOnly" (id 2) (at 183.515 152.4 0)
       (effects (font (size 1.27 1.27)) hide)
     )
@@
       (effects (font (size 1.27 1.27)) (justify left))
     )
-    (property "Footprint" "MountingHole:MountingHole_3mm_Pad_TopOnly" (id 2) (at 190.5 158.75 0)
+    (property "Footprint" "revxlp:MountingHole_3mm_Pad_NonPTH_TopOnly" (id 2) (at 190.5 158.75 0)
       (effects (font (size 1.27 1.27)) hide)
     )
@@
     )
     (path "/d668e699-ab17-4569-8fb7-e32e8aaed59e"
-      (reference "H1") (unit 1) (value "MountingHole") (footprint "MountingHole:MountingHole_3mm_Pad_TopOnly")
+      (reference "H1") (unit 1) (value "MountingHole") (footprint "revxlp:MountingHole_3mm_Pad_NonPTH_TopOnly")
     )
     (path "/50f54e4b-0933-4757-9ac9-2f865ea8908e"
-      (reference "H2") (unit 1) (value "MountingHole") (footprint "MountingHole:MountingHole_3mm_Pad_TopOnly")
+      (reference "H2") (unit 1) (value "MountingHole") (footprint "revxlp:MountingHole_3mm_Pad_NonPTH_TopOnly")
     )
     (path "/be5350c1-fa86-43a9-b1d8-e189608ad5ac"
-      (reference "H3") (unit 1) (value "MountingHole") (footprint "MountingHole:MountingHole_3mm_Pad_TopOnly")
+      (reference "H3") (unit 1) (value "MountingHole") (footprint "revxlp:MountingHole_3mm_Pad_NonPTH_TopOnly")
     )
     (path "/e89d20fd-de0f-4c68-89c7-445e7cb108d7"
-      (reference "H4") (unit 1) (value "MountingHole") (footprint "MountingHole:MountingHole_3mm_Pad_TopOnly")
+      (reference "H4") (unit 1) (value "MountingHole") (footprint "revxlp:MountingHole_3mm_Pad_NonPTH_TopOnly")
     )
     (path "/62f0725c-6ab8-4cb9-bc3d-061d4f32a171"
-      (reference "H5") (unit 1) (value "MountingHole") (footprint "MountingHole:MountingHole_3mm_Pad_TopOnly")
+      (reference "H5") (unit 1) (value "MountingHole") (footprint "revxlp:MountingHole_3mm_Pad_NonPTH_TopOnly")
     )
     (path "/87ebb9fd-6588-4af4-b1d3-9119acfaa6a6"
-      (reference "H6") (unit 1) (value "MountingHole") (footprint "MountingHole:MountingHole_3mm_Pad_TopOnly")
+      (reference "H6") (unit 1) (value "MountingHole") (footprint "revxlp:MountingHole_3mm_Pad_NonPTH_TopOnly")
+    )
+    (path "/6c3d5d6c-4e43-46bf-b738-d45a674e19ea"
+      (reference "H7") (unit 1) (value "MountingHole") (footprint "revxlp:MountingHole_3mm_Pad_NonPTH_TopOnly")
     )
     (path "/00000000-0000-0000-0000-00006075d32d"

Commit message: Reset/power tweaks, major silk improvements, etc.
* Move to different reset switch w/ better use w/ the case.
* Move the power slider to the edge for easier case access.
* Lots of silk improvements, tweaks, etc for controller and
  shift register area.
Parts:
- SW2: footprint revxlp:alps_sksn -> Button_Switch_SMD:Panasonic_EVQPUL_EVQPUC
Changed lines of the file:
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@@
     (property "Reference" "SW2" (id 0) (at 259.08 129.921 0))
     (property "Value" "SW_Push" (id 1) (at 259.08 132.2324 0))
-    (property "Footprint" "revxlp:alps_sksn" (id 2) (at 259.08 132.08 0)
+    (property "Footprint" "Button_Switch_SMD:Panasonic_EVQPUL_EVQPUC" (id 2) (at 259.08 132.08 0)
       (effects (font (size 1.27 1.27)) hide)
     )
@@
     )
     (path "/00000000-0000-0000-0000-0000608d2db9"
-      (reference "SW2") (unit 1) (value "SW_Push") (footprint "revxlp:alps_sksn")
+      (reference "SW2") (unit 1) (value "SW_Push") (footprint "Button_Switch_SMD:Panasonic_EVQPUL_EVQPUC")
     )
     (path "/00000000-0000-0000-0000-0000604dd518"

Commit message: Updated LCSC part numbers for LED resistors.
Parts:
- R_A0, R_A1, R_A2, R_A3, R_A4, R_A5, R_AltG2, R_B0, R_B1, R_B2, R_B3, R_B4, R_B5, R_C0, R_C1, R_C2, R_C3, R_C4, R_C5, R_D0, R_D1, R_D2, R_D3, R_D4, R_D5, R_E0, R_E1, R_E2, R_E3, R_E4, R_E5, R_F0, R_F1, R_F2, R_F3, R_F4, R_F5, R_G0, R_G1, R_G2, R_G3, R_G4, R_G5: LCSC Part Number (none) -> C17901
Changed lines of the file:
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@@
+      (effects (font (size 1.27 1.27)) hide)
+    )
+    (property "LCSC Part Number" "C17901" (id 4) (at 40.64 43.18 0)
       (effects (font (size 1.27 1.27)) hide)
     )
@@
       (effects (font (size 1.27 1.27)) hide)
     )
+    (property "LCSC Part Number" "C17901" (id 4) (at 40.64 43.18 0)
+      (effects (font (size 1.27 1.27)) hide)
+    )
     (pin "1")
     (pin "2")
@@
       (effects (font (size 1.27 1.27)) hide)
     )
+    (property "LCSC Part Number" "C17901" (id 4) (at 40.64 43.18 0)
+      (effects (font (size 1.27 1.27)) hide)
+    )
     (pin "1")
     (pin "2")
@@
       (effects (font (size 1.27 1.27)) hide)
     )
+    (property "LCSC Part Number" "C17901" (id 4) (at 40.64 43.18 0)
+      (effects (font (size 1.27 1.27)) hide)
+    )
     (pin "1")
     (pin "2")
@@
       (effects (font (size 1.27 1.27)) hide)
     )
+    (property "LCSC Part Number" "C17901" (id 4) (at 40.64 43.18 0)
+      (effects (font (size 1.27 1.27)) hide)
+    )
     (pin "1")
     (pin "2")
@@
       (effects (font (size 1.27 1.27)) hide)
     )
+    (property "LCSC Part Number" "C17901" (id 4) (at 40.64 43.18 0)
+      (effects (font (size 1.27 1.27)) hide)
+    )
     (pin "1")
     (pin "2")
@@
       (effects (font (size 1.27 1.27)) hide)
     )
+    (property "LCSC Part Number" "C17901" (id 4) (at 40.64 43.18 0)
+      (effects (font (size 1.27 1.27)) hide)
+    )
     (pin "1")
     (pin "2")
@@
       (effects (font (size 1.27 1.27)) hide)
     )
+    (property "LCSC Part Number" "C17901" (id 4) (at 40.64 43.18 0)
+      (effects (font (size 1.27 1.27)) hide)
+    )
     (pin "1")
     (pin "2")
@@
       (effects (font (size 1.27 1.27)) hide)
     )
+    (property "LCSC Part Number" "C17901" (id 4) (at 40.64 43.18 0)
+      (effects (font (size 1.27 1.27)) hide)
+    )
     (pin "1")
     (pin "2")
@@
       (effects (font (size 1.27 1.27)) hide)
     )
+    (property "LCSC Part Number" "C17901" (id 4) (at 40.64 43.18 0)
+      (effects (font (size 1.27 1.27)) hide)
+    )
     (pin "1")
     (pin "2")
@@
       (effects (font (size 1.27 1.27)) hide)
     )
+    (property "LCSC Part Number" "C17901" (id 4) (at 40.64 43.18 0)
+      (effects (font (size 1.27 1.27)) hide)
+    )
     (pin "1")
     (pin "2")
@@
       (effects (font (size 1.27 1.27)) hide)
     )
+    (property "LCSC Part Number" "C17901" (id 4) (at 40.64 43.18 0)
+      (effects (font (size 1.27 1.27)) hide)
+    )
     (pin "1")
     (pin "2")
@@
       (effects (font (size 1.27 1.27)) hide)
     )
+    (property "LCSC Part Number" "C17901" (id 4) (at 40.64 43.18 0)
+      (effects (font (size 1.27 1.27)) hide)
+    )
     (pin "1")
     (pin "2")
@@
       (effects (font (size 1.27 1.27)) hide)
     )
+    (property "LCSC Part Number" "C17901" (id 4) (at 40.64 43.18 0)
+      (effects (font (size 1.27 1.27)) hide)
+    )
     (pin "1")
     (pin "2")
@@
       (effects (font (size 1.27 1.27)) hide)
     )
+    (property "LCSC Part Number" "C17901" (id 4) (at 40.64 43.18 0)
+      (effects (font (size 1.27 1.27)) hide)
+    )
     (pin "1")
     (pin "2")
@@
       (effects (font (size 1.27 1.27)) hide)
     )
+    (property "LCSC Part Number" "C17901" (id 4) (at 40.64 43.18 0)
+      (effects (font (size 1.27 1.27)) hide)
+    )
     (pin "1")
     (pin "2")
@@
       (effects (font (size 1.27 1.27)) hide)
     )
+    (property "LCSC Part Number" "C17901" (id 4) (at 40.64 43.18 0)
+      (effects (font (size 1.27 1.27)) hide)
+    )
     (pin "1")
     (pin "2")
@@
       (effects (font (size 1.27 1.27)) hide)
     )
+    (property "LCSC Part Number" "C17901" (id 4) (at 40.64 43.18 0)
+      (effects (font (size 1.27 1.27)) hide)
+    )
     (pin "1")
     (pin "2")
@@
       (effects (font (size 1.27 1.27)) hide)
     )
+    (property "LCSC Part Number" "C17901" (id 4) (at 40.64 43.18 0)
+      (effects (font (size 1.27 1.27)) hide)
+    )
     (pin "1")
     (pin "2")
@@
       (effects (font (size 1.27 1.27)) hide)
     )
+    (property "LCSC Part Number" "C17901" (id 4) (at 40.64 43.18 0)
+      (effects (font (size 1.27 1.27)) hide)
+    )
     (pin "1")
     (pin "2")
@@
       (effects (font (size 1.27 1.27)) hide)
     )
+    (property "LCSC Part Number" "C17901" (id 4) (at 40.64 43.18 0)
+      (effects (font (size 1.27 1.27)) hide)
+    )
     (pin "1")
     (pin "2")
@@
       (effects (font (size 1.27 1.27)) hide)
     )
+    (property "LCSC Part Number" "C17901" (id 4) (at 40.64 43.18 0)
+      (effects (font (size 1.27 1.27)) hide)
+    )
     (pin "1")
     (pin "2")
@@
       (effects (font (size 1.27 1.27)) hide)
     )
+    (property "LCSC Part Number" "C17901" (id 4) (at 40.64 43.18 0)
+      (effects (font (size 1.27 1.27)) hide)
+    )
     (pin "1")
     (pin "2")
@@
       (effects (font (size 1.27 1.27)) hide)
     )
+    (property "LCSC Part Number" "C17901" (id 4) (at 40.64 43.18 0)
+      (effects (font (size 1.27 1.27)) hide)
+    )
     (pin "1")
     (pin "2")
@@
       (effects (font (size 1.27 1.27)) hide)
     )
+    (property "LCSC Part Number" "C17901" (id 4) (at 40.64 43.18 0)
+      (effects (font (size 1.27 1.27)) hide)
+    )
     (pin "1")
     (pin "2")
@@
       (effects (font (size 1.27 1.27)) hide)
     )
+    (property "LCSC Part Number" "C17901" (id 4) (at 40.64 43.18 0)
+      (effects (font (size 1.27 1.27)) hide)
+    )
     (pin "1")
     (pin "2")
@@
       (effects (font (size 1.27 1.27)) hide)
     )
+    (property "LCSC Part Number" "C17901" (id 4) (at 40.64 43.18 0)
+      (effects (font (size 1.27 1.27)) hide)
+    )
     (pin "1")
     (pin "2")
@@
       (effects (font (size 1.27 1.27)) hide)
     )
+    (property "LCSC Part Number" "C17901" (id 4) (at 40.64 43.18 0)
+      (effects (font (size 1.27 1.27)) hide)
+    )
     (pin "1")
     (pin "2")
@@
       (effects (font (size 1.27 1.27)) hide)
     )
+    (property "LCSC Part Number" "C17901" (id 4) (at 40.64 43.18 0)
+      (effects (font (size 1.27 1.27)) hide)
+    )
     (pin "1")
     (pin "2")
@@
       (effects (font (size 1.27 1.27)) hide)
     )
+    (property "LCSC Part Number" "C17901" (id 4) (at 40.64 43.18 0)
+      (effects (font (size 1.27 1.27)) hide)
+    )
     (pin "1")
     (pin "2")
@@
       (effects (font (size 1.27 1.27)) hide)
     )
+    (property "LCSC Part Number" "C17901" (id 4) (at 40.64 43.18 0)
+      (effects (font (size 1.27 1.27)) hide)
+    )
     (pin "1")
     (pin "2")
@@
       (effects (font (size 1.27 1.27)) hide)
     )
+    (property "LCSC Part Number" "C17901" (id 4) (at 40.64 43.18 0)
+      (effects (font (size 1.27 1.27)) hide)
+    )
     (pin "1")
     (pin "2")
@@
       (effects (font (size 1.27 1.27)) hide)
     )
+    (property "LCSC Part Number" "C17901" (id 4) (at 40.64 43.18 0)
+      (effects (font (size 1.27 1.27)) hide)
+    )
     (pin "1")
     (pin "2")
@@
       (effects (font (size 1.27 1.27)) hide)
     )
+    (property "LCSC Part Number" "C17901" (id 4) (at 40.64 43.18 0)
+      (effects (font (size 1.27 1.27)) hide)
+    )
     (pin "1")
     (pin "2")
@@
       (effects (font (size 1.27 1.27)) hide)
     )
+    (property "LCSC Part Number" "C17901" (id 4) (at 40.64 43.18 0)
+      (effects (font (size 1.27 1.27)) hide)
+    )
     (pin "1")
     (pin "2")
@@
       (effects (font (size 1.27 1.27)) hide)
     )
+    (property "LCSC Part Number" "C17901" (id 4) (at 40.64 43.18 0)
+      (effects (font (size 1.27 1.27)) hide)
+    )
     (pin "1")
     (pin "2")
@@
       (effects (font (size 1.27 1.27)) hide)
     )
+    (property "LCSC Part Number" "C17901" (id 4) (at 40.64 43.18 0)
+      (effects (font (size 1.27 1.27)) hide)
+    )
     (pin "1")
     (pin "2")
@@
       (effects (font (size 1.27 1.27)) hide)
     )
+    (property "LCSC Part Number" "C17901" (id 4) (at 40.64 43.18 0)
+      (effects (font (size 1.27 1.27)) hide)
+    )
     (pin "1")
     (pin "2")
@@
       (effects (font (size 1.27 1.27)) hide)
     )
+    (property "LCSC Part Number" "C17901" (id 4) (at 40.64 43.18 0)
+      (effects (font (size 1.27 1.27)) hide)
+    )
     (pin "1")
     (pin "2")
@@
       (effects (font (size 1.27 1.27)) hide)
     )
+    (property "LCSC Part Number" "C17901" (id 4) (at 40.64 43.18 0)
+      (effects (font (size 1.27 1.27)) hide)
+    )
     (pin "1")
     (pin "2")
@@
       (effects (font (size 1.27 1.27)) hide)
     )
+    (property "LCSC Part Number" "C17901" (id 4) (at 40.64 43.18 0)
+      (effects (font (size 1.27 1.27)) hide)
+    )
     (pin "1")
     (pin "2")
@@
     )
     (property "Datasheet" "~" (id 3) (at 163.83 167.64 0)
+      (effects (font (size 1.27 1.27)) hide)
+    )
+    (property "LCSC Part Number" "C17901" (id 4) (at 40.64 43.18 0)
       (effects (font (size 1.27 1.27)) hide)
     )
@@
       (effects (font (size 1.27 1.27)) hide)
     )
+    (property "LCSC Part Number" "C17901" (id 4) (at 40.64 43.18 0)
+      (effects (font (size 1.27 1.27)) hide)
+    )
