File: pcb/revxlp.kicad_sch (KiCad schematic)
At the start: 144 parts, among them Q1 AO3416 N-channel MOSFET, SW1 SW_SPDT, SW2 SW_Push, U1 74HC595, U2 SeeeduinoXIAO_BLE

Commit message: Reset/power silk, mounting hole PCBA fixes.
Parts:
- H1, H2, H3, H4, H5, H6, H7: LCSC Part Number (none) -> C2915634
- SW1: footprint revxlp:switch_SSSS811101 -> Button_Switch_SMD:SW_SPDT_PCM12; LCSC Part Number (none) -> C221841
- SW2: LCSC Part Number (none) -> C79174
Changed lines of the file:
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@@
     (property "Reference" "SW1" (id 0) (at 255.27 146.05 0))
     (property "Value" "SW_SPDT" (id 1) (at 255.27 148.59 0))
-    (property "Footprint" "revxlp:switch_SSSS811101" (id 2) (at 256.54 152.4 0)
+    (property "Footprint" "Button_Switch_SMD:SW_SPDT_PCM12" (id 2) (at 256.54 152.4 0)
       (effects (font (size 1.27 1.27)) hide)
     )
@@
       (effects (font (size 1.27 1.27)) hide)
     )
+    (property "LCSC Part Number" "C221841" (id 4) (at 256.54 152.4 0)
+      (effects (font (size 1.27 1.27)) hide)
+    )
     (pin "1")
     (pin "2")
@@
       (effects (font (size 1.27 1.27)) hide)
     )
+    (property "LCSC Part Number" "C79174" (id 4) (at 259.08 137.16 0)
+      (effects (font (size 1.27 1.27)) hide)
+    )
     (pin "1")
     (pin "2")
@@
       (effects (font (size 1.27 1.27)) hide)
     )
+    (property "LCSC Part Number" "C2915634" (id 4) (at 183.515 152.4 0)
+      (effects (font (size 1.27 1.27)) hide)
+    )
   )
   (symbol (lib_id "Mechanical:MountingHole") (at 213.995 158.75 0) (unit 1)
@@
       (effects (font (size 1.27 1.27)) hide)
     )
+    (property "LCSC Part Number" "C2915634" (id 4) (at 183.515 152.4 0)
+      (effects (font (size 1.27 1.27)) hide)
+    )
   )
   (symbol (lib_id "Seeeduino XIAO:SeeeduinoXIAO_BLE") (at 227.33 49.53 0) (unit 1)
@@
       (effects (font (size 1.27 1.27)) hide)
     )
+    (property "LCSC Part Number" "C2915634" (id 4) (at 183.515 152.4 0)
+      (effects (font (size 1.27 1.27)) hide)
+    )
   )
   (symbol (lib_id "power:+3V3") (at 207.01 95.885 0) (unit 1)
@@
       (effects (font (size 1.27 1.27)) hide)
     )
+    (property "LCSC Part Number" "C2915634" (id 4) (at 183.515 152.4 0)
+      (effects (font (size 1.27 1.27)) hide)
+    )
   )
   (symbol (lib_name "Battery_Cell_1") (lib_id "Device:Battery_Cell") (at 269.24 161.29 270) (unit 1)
@@
       (effects (font (size 1.27 1.27)) hide)
     )
+    (property "LCSC Part Number" "C2915634" (id 4) (at 183.515 152.4 0)
+      (effects (font (size 1.27 1.27)) hide)
+    )
   )
   (symbol (lib_id "Mechanical:MountingHole") (at 183.515 152.4 0) (unit 1)
@@
       (effects (font (size 1.27 1.27)) hide)
     )
+    (property "LCSC Part Number" "C2915634" (id 4) (at 183.515 152.4 0)
+      (effects (font (size 1.27 1.27)) hide)
+    )
   )
   (symbol (lib_id "Device:R_Small_US") (at 99.695 189.865 180) (unit 1)
@@
       (effects (font (size 1.27 1.27)) hide)
     )
+    (property "LCSC Part Number" "C2915634" (id 4) (at 183.515 152.4 0)
+      (effects (font (size 1.27 1.27)) hide)
+    )
   )
   (symbol (lib_id "Switch:SW_Push_LED") (at 104.775 184.785 0) (unit 1)
@@
     )
     (path "/00000000-0000-0000-0000-0000606f98ae"
-      (reference "SW1") (unit 1) (value "SW_SPDT") (footprint "revxlp:switch_SSSS811101")
+      (reference "SW1") (unit 1) (value "SW_SPDT") (footprint "Button_Switch_SMD:SW_SPDT_PCM12")
     )
     (path "/00000000-0000-0000-0000-0000608d2db9"

Commit message: Better case, debugging w/ assembly, 2mm solder nuts.
Parts:
- H1, H2, H3, H4, H5, H6, H7: LCSC Part Number C2915634 -> C2916381
Changed lines of the file:
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@@
       (effects (font (size 1.27 1.27)) hide)
     )
-    (property "LCSC Part Number" "C2915634" (id 4) (at 183.515 152.4 0)
+    (property "LCSC Part Number" "C2916381" (id 4) (at 183.515 152.4 0)
       (effects (font (size 1.27 1.27)) hide)
     )
@@
       (effects (font (size 1.27 1.27)) hide)
     )
-    (property "LCSC Part Number" "C2915634" (id 4) (at 183.515 152.4 0)
+    (property "LCSC Part Number" "C2916381" (id 4) (at 183.515 152.4 0)
       (effects (font (size 1.27 1.27)) hide)
     )
@@
       (effects (font (size 1.27 1.27)) hide)
     )
-    (property "LCSC Part Number" "C2915634" (id 4) (at 183.515 152.4 0)
+    (property "LCSC Part Number" "C2916381" (id 4) (at 183.515 152.4 0)
       (effects (font (size 1.27 1.27)) hide)
     )
@@
       (effects (font (size 1.27 1.27)) hide)
     )
-    (property "LCSC Part Number" "C2915634" (id 4) (at 183.515 152.4 0)
+    (property "LCSC Part Number" "C2916381" (id 4) (at 183.515 152.4 0)
       (effects (font (size 1.27 1.27)) hide)
     )
@@
       (effects (font (size 1.27 1.27)) hide)
     )
-    (property "LCSC Part Number" "C2915634" (id 4) (at 183.515 152.4 0)
+    (property "LCSC Part Number" "C2916381" (id 4) (at 183.515 152.4 0)
       (effects (font (size 1.27 1.27)) hide)
     )
@@
       (effects (font (size 1.27 1.27)) hide)
     )
-    (property "LCSC Part Number" "C2915634" (id 4) (at 183.515 152.4 0)
+    (property "LCSC Part Number" "C2916381" (id 4) (at 183.515 152.4 0)
       (effects (font (size 1.27 1.27)) hide)
     )
@@
       (effects (font (size 1.27 1.27)) hide)
     )
-    (property "LCSC Part Number" "C2915634" (id 4) (at 183.515 152.4 0)
-      (effects (font (size 1.27 1.27)) hide)
-    )
+    (property "LCSC Part Number" "C2916381" (id 4) (at 183.515 152.4 0)
+      (effects (font (size 1.27 1.27)) hide)
+    )

Commit message: Move to M2 mounting hardware.
* New M2 footprint.
* Switch to M2 LCSC part number.
* Smaller holes in the case.
* Adjust the bottom plate hole size.
Parts:
- H1, H2, H3, H4, H5, H6, H7: LCSC Part Number C2916381 -> C2915626
Changed lines of the file:
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@@
       (effects (font (size 1.27 1.27)) hide)
     )
-    (property "LCSC Part Number" "C2916381" (id 4) (at 183.515 152.4 0)
+    (property "LCSC Part Number" "C2915626" (id 4) (at 183.515 152.4 0)
       (effects (font (size 1.27 1.27)) hide)
     )
@@
       (effects (font (size 1.27 1.27)) hide)
     )
-    (property "LCSC Part Number" "C2916381" (id 4) (at 183.515 152.4 0)
+    (property "LCSC Part Number" "C2915626" (id 4) (at 183.515 152.4 0)
       (effects (font (size 1.27 1.27)) hide)
     )
@@
       (effects (font (size 1.27 1.27)) hide)
     )
-    (property "LCSC Part Number" "C2916381" (id 4) (at 183.515 152.4 0)
+    (property "LCSC Part Number" "C2915626" (id 4) (at 183.515 152.4 0)
       (effects (font (size 1.27 1.27)) hide)
     )
@@
       (effects (font (size 1.27 1.27)) hide)
     )
-    (property "LCSC Part Number" "C2916381" (id 4) (at 183.515 152.4 0)
+    (property "LCSC Part Number" "C2915626" (id 4) (at 183.515 152.4 0)
       (effects (font (size 1.27 1.27)) hide)
     )
@@
       (effects (font (size 1.27 1.27)) hide)
     )
-    (property "LCSC Part Number" "C2916381" (id 4) (at 183.515 152.4 0)
+    (property "LCSC Part Number" "C2915626" (id 4) (at 183.515 152.4 0)
       (effects (font (size 1.27 1.27)) hide)
     )
@@
       (effects (font (size 1.27 1.27)) hide)
     )
-    (property "LCSC Part Number" "C2916381" (id 4) (at 183.515 152.4 0)
+    (property "LCSC Part Number" "C2915626" (id 4) (at 183.515 152.4 0)
       (effects (font (size 1.27 1.27)) hide)
     )
@@
       (effects (font (size 1.27 1.27)) hide)
     )
-    (property "LCSC Part Number" "C2916381" (id 4) (at 183.515 152.4 0)
-      (effects (font (size 1.27 1.27)) hide)
-    )
+    (property "LCSC Part Number" "C2915626" (id 4) (at 183.515 152.4 0)
+      (effects (font (size 1.27 1.27)) hide)
+    )
