File: plate/revxlp_plate.kicad_pcb (KiCad board)
At the start: 2 copper layers, 238.7 x 89.1 mm, 2 parts

Commit message: Better plate corner by the controller.
Parts:
- moved REF** 32.8 mm to (154.0, 91.5)
- moved rev41lp_edgecutSwitchPlate 32.8 mm to (154.2, 28.8)
Other:
- outline, holes or cut-outs redrawn
- board text added: "revxlp : v0.1 : 2022/10"
- board text removed: "revxlp : v0.1 : 2022/04"
