File: bottom/revxlp_bottom.kicad_pcb (KiCad board)
At the start: 2 copper layers, 238.7 x 94.8 mm, 9 parts

Commit message: Add bumpon insets to case.
Parts:
- added BMP1: Bumpon, revxlp:Bumpon, F.Cu at (49.7, 33.2)
- added BMP2: Bumpon, revxlp:Bumpon, F.Cu at (259.1, 32.9)
- added BMP3: Bumpon, revxlp:Bumpon, F.Cu at (39.7, 75.1)
- added BMP4: Bumpon, revxlp:Bumpon, F.Cu at (268.6, 75.1)
- added BMP5: Bumpon, revxlp:Bumpon, F.Cu at (118.7, 107.5)
- added BMP6: Bumpon, revxlp:Bumpon, F.Cu at (190.1, 107.5)
Changed lines of the file:
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@@
     (fp_line (start -40.441671 77.515789) (end -39.503394 81.579917) (layer "Edge.Cuts") (width 0.2))
     (fp_arc (start 40.441672 77.515789) (mid 40.793521 76.958127) (end 41.416042 76.74074) (layer "Edge.Cuts") (width 0.2))
-    (fp_arc (start 49.460861 0.512599) (mid 51.695817 0.128561) (end 53.959882 0) (layer "Edge.Cuts") (width 0.2))
+    (fp_arc (start 49.460861 0.512599) (mid 51.695817 0.128555) (end 53.959882 0) (layer "Edge.Cuts") (width 0.2))
     (fp_arc (start -7.200363 -7.073925) (mid -6.757044 -7.696834) (end -6.003106 -7.823822) (layer "Edge.Cuts") (width 0.2))
     (fp_arc (start -84.840673 53.741991) (mid -82.576609 53.870554) (end -80.341652 54.25459) (layer "Edge.Cuts") (width 0.2))
     (fp_arc (start -16.510921 86.938468) (mid -18.774985 86.809905) (end -21.009942 86.425869) (layer "Edge.Cuts") (width 0.2))
-    (fp_arc (start 39.503394 81.579917) (mid 39.236784 82.062735) (end 38.753975 82.329336) (layer "Edge.Cuts") (width 0.2))
+    (fp_arc (start 39.503394 81.579917) (mid 39.236846 82.062797) (end 38.753975 82.329336) (layer "Edge.Cuts") (width 0.2))
     (fp_arc (start -10.776776 8.41722) (mid -11.221228 9.040317) (end -11.976099 9.166638) (layer "Edge.Cuts") (width 0.2))
     (fp_arc (start 56.605052 60.530052) (mid 56.822458 59.907551) (end 57.380101 59.555682) (layer "Edge.Cuts") (width 0.2))
@@
     (fp_arc (start 56.605052 75.74074) (mid 56.31206 76.447752) (end 55.605051 76.74074) (layer "Edge.Cuts") (width 0.2))
     (fp_arc (start -118.574096 49.692873) (mid -119.197193 49.248422) (end -119.323515 48.493552) (layer "Edge.Cuts") (width 0.2))
-    (fp_arc (start 103.255743 53.229393) (mid 101.020786 53.613425) (end 98.756722 53.741991) (layer "Edge.Cuts") (width 0.2))
+    (fp_arc (start 103.255743 53.229393) (mid 101.020786 53.613422) (end 98.756722 53.741991) (layer "Edge.Cuts") (width 0.2))
     (fp_arc (start -57.380101 59.555682) (mid -56.822443 59.907537) (end -56.605052 60.530052) (layer "Edge.Cuts") (width 0.2))
     (fp_arc (start -108.30683 0.775049) (mid -107.954975 0.217391) (end -107.33246 0) (layer "Edge.Cuts") (width 0.2))
@@
     (fp_arc (start 119.323515 48.493552) (mid 119.197193 49.248429) (end 118.574096 49.692873) (layer "Edge.Cuts") (width 0.2))
   )
+  (footprint "revxlp:Bumpon" (layer "F.Cu")
+    (at 190.067222 107.481219)
+    (fp_text reference "BMP6" (at 0 -0.5 unlocked) (layer "F.SilkS")
+      (effects (font (size 1 1) (thickness 0.15)))
+    )
+    (fp_text value "Bumpon" (at 0 1 unlocked) (layer "F.Fab")
+      (effects (font (size 1 1) (thickness 0.15)))
+    )
+    (fp_circle (center 0 0) (end 3.2 0) (layer "B.CrtYd") (width 0.12) (fill none))
+  )
+  (footprint "revxlp:Bumpon" (layer "F.Cu")
+    (at 39.692222 75.081219)
+    (fp_text reference "BMP3" (at 0 -0.5 unlocked) (layer "F.SilkS")
+      (effects (font (size 1 1) (thickness 0.15)))
+    )
+    (fp_text value "Bumpon" (at 0 1 unlocked) (layer "F.Fab")
+      (effects (font (size 1 1) (thickness 0.15)))
+    )
+    (fp_circle (center 0 0) (end 3.2 0) (layer "B.CrtYd") (width 0.12) (fill none))
+  )
+  (footprint "revxlp:Bumpon" (layer "F.Cu")
+    (at 259.067222 32.881219)
+    (fp_text reference "BMP2" (at 0 -0.5 unlocked) (layer "F.SilkS")
+      (effects (font (size 1 1) (thickness 0.15)))
+    )
+    (fp_text value "Bumpon" (at 0 1 unlocked) (layer "F.Fab")
+      (effects (font (size 1 1) (thickness 0.15)))
+    )
+    (fp_circle (center 0 0) (end 3.2 0) (layer "B.CrtYd") (width 0.12) (fill none))
+  )
+  (footprint "revxlp:Bumpon" (layer "F.Cu")
+    (at 268.592222 75.081219)
+    (fp_text reference "BMP4" (at 0 -0.5 unlocked) (layer "F.SilkS")
+      (effects (font (size 1 1) (thickness 0.15)))
+    )
+    (fp_text value "Bumpon" (at 0 1 unlocked) (layer "F.Fab")
+      (effects (font (size 1 1) (thickness 0.15)))
+    )
+    (fp_circle (center 0 0) (end 3.2 0) (layer "B.CrtYd") (width 0.12) (fill none))
+  )
+  (footprint "revxlp:Bumpon" (layer "F.Cu")
+    (at 118.742222 107.456219)
+    (fp_text reference "BMP5" (at 0 -0.5 unlocked) (layer "F.SilkS")
+      (effects (font (size 1 1) (thickness 0.15)))
+    )
+    (fp_text value "Bumpon" (at 0 1 unlocked) (layer "F.Fab")
+      (effects (font (size 1 1) (thickness 0.15)))
+    )
+    (fp_circle (center 0 0) (end 3.2 0) (layer "B.CrtYd") (width 0.12) (fill none))
+  )
+  (footprint "revxlp:Bumpon" (layer "F.Cu")
+    (at 49.667222 33.206219)
+    (fp_text reference "BMP1" (at 0 -0.5 unlocked) (layer "F.SilkS")
+      (effects (font (size 1 1) (thickness 0.15)))
+    )
+    (fp_text value "Bumpon" (at 0 1 unlocked) (layer "F.Fab")
+      (effects (font (size 1 1) (thickness 0.15)))
+    )
+    (fp_circle (center 0 0) (end 3.2 0) (layer "B.CrtYd") (width 0.12) (fill none))
+  )
   (footprint "MountingHole:MountingHole_3mm" (layer "B.Cu")

Commit message: Fix bottom plate silk location, add additional bumpon.
Parts:
- added BMP2: Bumpon, revxlp:Bumpon, F.Cu at (154.2, 38.4)
- moved G*** 34.3 mm to (154.1, 31.3)
- renumbered BMP2 to BMP3, BMP3 to BMP4, BMP4 to BMP5, BMP5 to BMP6, BMP6 to BMP7
Changed lines of the file:
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@@
     (fp_line (start -40.441671 77.515789) (end -39.503394 81.579917) (layer "Edge.Cuts") (width 0.2))
     (fp_arc (start 40.441672 77.515789) (mid 40.793521 76.958127) (end 41.416042 76.74074) (layer "Edge.Cuts") (width 0.2))
-    (fp_arc (start 49.460861 0.512599) (mid 51.695817 0.128555) (end 53.959882 0) (layer "Edge.Cuts") (width 0.2))
+    (fp_arc (start 49.460861 0.512599) (mid 51.695817 0.128561) (end 53.959882 0) (layer "Edge.Cuts") (width 0.2))
     (fp_arc (start -7.200363 -7.073925) (mid -6.757044 -7.696834) (end -6.003106 -7.823822) (layer "Edge.Cuts") (width 0.2))
     (fp_arc (start -84.840673 53.741991) (mid -82.576609 53.870554) (end -80.341652 54.25459) (layer "Edge.Cuts") (width 0.2))
     (fp_arc (start -16.510921 86.938468) (mid -18.774985 86.809905) (end -21.009942 86.425869) (layer "Edge.Cuts") (width 0.2))
-    (fp_arc (start 39.503394 81.579917) (mid 39.236846 82.062797) (end 38.753975 82.329336) (layer "Edge.Cuts") (width 0.2))
+    (fp_arc (start 39.503394 81.579917) (mid 39.236861 82.062812) (end 38.753975 82.329336) (layer "Edge.Cuts") (width 0.2))
     (fp_arc (start -10.776776 8.41722) (mid -11.221228 9.040317) (end -11.976099 9.166638) (layer "Edge.Cuts") (width 0.2))
     (fp_arc (start 56.605052 60.530052) (mid 56.822458 59.907551) (end 57.380101 59.555682) (layer "Edge.Cuts") (width 0.2))
@@
     (fp_arc (start 56.605052 75.74074) (mid 56.31206 76.447752) (end 55.605051 76.74074) (layer "Edge.Cuts") (width 0.2))
     (fp_arc (start -118.574096 49.692873) (mid -119.197193 49.248422) (end -119.323515 48.493552) (layer "Edge.Cuts") (width 0.2))
-    (fp_arc (start 103.255743 53.229393) (mid 101.020786 53.613422) (end 98.756722 53.741991) (layer "Edge.Cuts") (width 0.2))
+    (fp_arc (start 103.255743 53.229393) (mid 101.020786 53.613423) (end 98.756722 53.741991) (layer "Edge.Cuts") (width 0.2))
     (fp_arc (start -57.380101 59.555682) (mid -56.822443 59.907537) (end -56.605052 60.530052) (layer "Edge.Cuts") (width 0.2))
     (fp_arc (start -108.30683 0.775049) (mid -107.954975 0.217391) (end -107.33246 0) (layer "Edge.Cuts") (width 0.2))
-    (fp_arc (start 40.244726 2.638295) (mid 39.79442 2.693222) (end 39.343321 2.645225) (layer "Edge.Cuts") (width 0.2))
+    (fp_arc (start 40.244726 2.638295) (mid 39.794418 2.693234) (end 39.343321 2.645225) (layer "Edge.Cuts") (width 0.2))
     (fp_arc (start -98.756723 53.741992) (mid -101.020787 53.613429) (end -103.255744 53.229393) (layer "Edge.Cuts") (width 0.2))
     (fp_arc (start -38.753975 82.329336) (mid -39.236131 82.062073) (end -39.503394 81.579917) (layer "Edge.Cuts") (width 0.2))
     (fp_arc (start -41.416042 76.740739) (mid -40.793527 76.958131) (end -40.441671 77.515789) (layer "Edge.Cuts") (width 0.2))
-    (fp_arc (start 107.332459 0) (mid 107.954995 0.217376) (end 108.30683 0.775048) (layer "Edge.Cuts") (width 0.2))
+    (fp_arc (start 107.332459 0) (mid 107.954971 0.217385) (end 108.30683 0.775048) (layer "Edge.Cuts") (width 0.2))
     (fp_arc (start -55.605052 76.74074) (mid -56.312159 76.447847) (end -56.605052 75.74074) (layer "Edge.Cuts") (width 0.2))
     (fp_arc (start 21.009942 86.425869) (mid 18.774985 86.809904) (end 16.510921 86.938468) (layer "Edge.Cuts") (width 0.2))
-    (fp_arc (start 119.323515 48.493552) (mid 119.197193 49.248429) (end 118.574096 49.692873) (layer "Edge.Cuts") (width 0.2))
+    (fp_arc (start 119.323515 48.493552) (mid 119.19719 49.24841) (end 118.574096 49.692873) (layer "Edge.Cuts") (width 0.2))
   )
   (footprint "revxlp:Bumpon" (layer "F.Cu")
     (at 190.067222 107.481219)
-    (fp_text reference "BMP6" (at 0 -0.5 unlocked) (layer "F.SilkS")
+    (fp_text reference "BMP7" (at 0 -0.5 unlocked) (layer "F.SilkS")
       (effects (font (size 1 1) (thickness 0.15)))
     )
@@
   (footprint "revxlp:Bumpon" (layer "F.Cu")
     (at 39.692222 75.081219)
+    (fp_text reference "BMP4" (at 0 -0.5 unlocked) (layer "F.SilkS")
+      (effects (font (size 1 1) (thickness 0.15)))
+    )
+    (fp_text value "Bumpon" (at 0 1 unlocked) (layer "F.Fab")
+      (effects (font (size 1 1) (thickness 0.15)))
+    )
+    (fp_circle (center 0 0) (end 3.2 0) (layer "B.CrtYd") (width 0.12) (fill none))
+  )
+  (footprint "revxlp:Bumpon" (layer "F.Cu")
+    (at 259.067222 32.881219)
     (fp_text reference "BMP3" (at 0 -0.5 unlocked) (layer "F.SilkS")
       (effects (font (size 1 1) (thickness 0.15)))
@@
   )
   (footprint "revxlp:Bumpon" (layer "F.Cu")
-    (at 259.067222 32.881219)
-    (fp_text reference "BMP2" (at 0 -0.5 unlocked) (layer "F.SilkS")
-      (effects (font (size 1 1) (thickness 0.15)))
-    )
-    (fp_text value "Bumpon" (at 0 1 unlocked) (layer "F.Fab")
-      (effects (font (size 1 1) (thickness 0.15)))
-    )
-    (fp_circle (center 0 0) (end 3.2 0) (layer "B.CrtYd") (width 0.12) (fill none))
-  )
-  (footprint "revxlp:Bumpon" (layer "F.Cu")
     (at 268.592222 75.081219)
-    (fp_text reference "BMP4" (at 0 -0.5 unlocked) (layer "F.SilkS")
+    (fp_text reference "BMP5" (at 0 -0.5 unlocked) (layer "F.SilkS")
       (effects (font (size 1 1) (thickness 0.15)))
     )
@@
   (footprint "revxlp:Bumpon" (layer "F.Cu")
     (at 118.742222 107.456219)
-    (fp_text reference "BMP5" (at 0 -0.5 unlocked) (layer "F.SilkS")
+    (fp_text reference "BMP6" (at 0 -0.5 unlocked) (layer "F.SilkS")
       (effects (font (size 1 1) (thickness 0.15)))
     )
@@
     (at 49.667222 33.206219)
     (fp_text reference "BMP1" (at 0 -0.5 unlocked) (layer "F.SilkS")
+      (effects (font (size 1 1) (thickness 0.15)))
+    )
+    (fp_text value "Bumpon" (at 0 1 unlocked) (layer "F.Fab")
+      (effects (font (size 1 1) (thickness 0.15)))
+    )
+    (fp_circle (center 0 0) (end 3.2 0) (layer "B.CrtYd") (width 0.12) (fill none))
+  )
+  (footprint "revxlp:Bumpon" (layer "F.Cu")
+    (at 154.229537 38.406219)
+    (fp_text reference "BMP2" (at 0 -0.5 unlocked) (layer "F.SilkS")
       (effects (font (size 1 1) (thickness 0.15)))
     )
@@
   )
   (footprint "revxlp:Z_Towel_Logo" (layer "B.Cu")
-    (at 155.588481 65.530604 -103)
+    (at 154.101067 31.255604 -103)
     (attr through_hole)
     (fp_text reference "G***" (at 0 0 77) (layer "B.SilkS") hide
