File: 12u/pcb/revxlp.kicad_sch (KiCad schematic)
At the start: 144 parts, among them Q1 AO3416 N-channel MOSFET, SW1 SW_SPDT, SW2 SW_Push, U1 74HC595, U2 SeeeduinoXIAO_BLE

Commit message: first commit
Parts:
- added OUTLINE1: Board outline, revxlp:rev41lp_edgecutBottomPlate, symbol revxlp:Board_Outline
- BT1: symbol Device:Battery_Cell -> revxlp:Battery_Cell; 10u-bottom:Footprint (none) -> revxlp:empty; 10u-top:Footprint (none) -> revxlp:empty; 10u:Footprint (none) -> revxlp:cell_pads; Config (none) -> +10u; bottom:Footprint (none) -> revxlp:empty; top:Footprint (none) -> revxlp:empty
- BT2: symbol Device:Battery_Cell -> revxlp:Battery_Cell_1; 10u-bottom:Footprint (none) -> revxlp:empty; 10u-top:Footprint (none) -> revxlp:empty; 10u:Footprint (none) -> Connector_JST:JST_SH_SM02B-SRSS-TB_1x02-1MP_P1.00mm_Horizon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; Config (none) -> +10u; bottom:Footprint (none) -> revxlp:empty; top:Footprint (none) -> revxlp:empty
- D_A0, D_B0, D_C0, D_D0, D_E0, D_F0: symbol Device:D -> revxlp:D; 10u-bottom:Footprint (none) -> revxlp:empty; 10u-top:Footprint (none) -> revxlp:empty; 10u:Footprint (none) -> revxlp:empty; Config (none) -> +10u; bottom:Footprint (none) -> revxlp:empty; top:Footprint (none) -> revxlp:empty
- D_A1, D_A2, D_A3, D_A4, D_A5, D_B1, D_B2, D_B3, D_B4, D_B5, D_C1, D_C2, D_C3, D_C4, D_C5, D_D1, D_D2, D_D3, D_D4, D_D5, D_E1, D_E2, D_E3, D_E4, D_E5, D_F1, D_F2, D_F3, D_F4, D_F5, D_G0, D_G1, D_G2, D_G3, D_G4, D_G5: symbol Device:D -> revxlp:D; 10u-bottom:Footprint (none) -> revxlp:empty; 10u-top:Footprint (none) -> revxlp:empty; 10u:Footprint (none) -> Diode_SMD:D_1206_3216Metric_Pad1.42x1.75mm_HandSolder; Config (none) -> +10u; bottom:Footprint (none) -> revxlp:empty; top:Footprint (none) -> revxlp:empty
- H1, H2, H3, H4, H5, H6, H7: symbol Mechanical:MountingHole -> revxlp:MountingHole; 10u-bottom:Footprint (none) -> revxlp:MountingHole_3mm_Pad_NonPTH_TopOnly; 10u-top:Footprint (none) -> revxlp:empty; 10u:Footprint (none) -> revxlp:MountingHole_3mm_Pad_NonPTH_TopOnly; Config (none) -> +bottom, +10u, +10u-bottom; bottom:Footprint (none) -> revxlp:MountingHole_3mm_Pad_NonPTH_TopOnly; top:Footprint (none) -> revxlp:empty
- JP1: symbol 41_1350_pcb-rescue:SolderJumper_3_Open-Jumper -> revxlp:SolderJumper_3_Open-Jumper; 10u-bottom:Footprint (none) -> revxlp:empty; 10u-top:Footprint (none) -> revxlp:empty; 10u:Footprint (none) -> Jumper:SolderJumper-3_P1.3mm_Open_RoundedPad1.0x1.5mm; Config (none) -> +10u; bottom:Footprint (none) -> revxlp:empty; top:Footprint (none) -> revxlp:empty
- Q1: symbol Device:Q_NMOS_GSD -> revxlp:Q_NMOS_GSD; 10u-bottom:Footprint (none) -> revxlp:empty; 10u-top:Footprint (none) -> revxlp:empty; 10u:Footprint (none) -> Package_TO_SOT_SMD:SOT-23; Config (none) -> +10u; bottom:Footprint (none) -> revxlp:empty; top:Footprint (none) -> revxlp:empty
- R80: symbol Device:R_US -> revxlp:R_US; 10u-bottom:Footprint (none) -> revxlp:empty; 10u-top:Footprint (none) -> revxlp:empty; 10u:Footprint (none) -> revxlp:empty; Config (none) -> +10u; bottom:Footprint (none) -> revxlp:empty; top:Footprint (none) -> revxlp:empty
- R_A0, R_B0, R_C0, R_D0, R_E0, R_F0: symbol Device:R_Small_US -> revxlp:R_Small_US; 10u-bottom:Footprint (none) -> revxlp:empty; 10u-top:Footprint (none) -> revxlp:empty; 10u:Footprint (none) -> revxlp:empty; Config (none) -> +10u; bottom:Footprint (none) -> revxlp:empty; top:Footprint (none) -> revxlp:empty
- R_A1, R_A2, R_A3, R_A4, R_A5, R_AltG2, R_B1, R_B2, R_B3, R_B4, R_B5, R_C1, R_C2, R_C3, R_C4, R_C5, R_D1, R_D2, R_D3, R_D4, R_D5, R_E1, R_E2, R_E3, R_E4, R_E5, R_F1, R_F2, R_F3, R_F4, R_F5, R_G0, R_G1, R_G2, R_G3, R_G4, R_G5: symbol Device:R_Small_US -> revxlp:R_Small_US; 10u-bottom:Footprint (none) -> revxlp:empty; 10u-top:Footprint (none) -> revxlp:empty; 10u:Footprint (none) -> Resistor_SMD:R_1206_3216Metric_Pad1.30x1.75mm_HandSolder; Config (none) -> +10u; bottom:Footprint (none) -> revxlp:empty; top:Footprint (none) -> revxlp:empty
- SW1: symbol Switch:SW_SPDT -> revxlp:SW_SPDT; 10u-bottom:Footprint (none) -> revxlp:empty; 10u-top:Footprint (none) -> revxlp:empty; 10u:Footprint (none) -> Button_Switch_SMD:SW_SPDT_PCM12; Config (none) -> +10u; bottom:Footprint (none) -> revxlp:empty; top:Footprint (none) -> revxlp:empty
- SW2: symbol Switch:SW_Push -> revxlp:SW_Push; 10u-bottom:Footprint (none) -> revxlp:empty; 10u-top:Footprint (none) -> revxlp:empty; 10u:Footprint (none) -> Button_Switch_SMD:Panasonic_EVQPUL_EVQPUC; Config (none) -> +10u; bottom:Footprint (none) -> revxlp:empty; top:Footprint (none) -> revxlp:empty
- SwA0, SwB0, SwC0, SwD0, SwE0, SwF0: symbol Switch:SW_Push_LED -> revxlp:SW_Push_LED; 10u-bottom:Footprint (none) -> revxlp:empty; 10u-top:Footprint (none) -> revxlp:pg1350_plate_cut; 10u:Footprint (none) -> revxlp:empty; Config (none) -> +top, +10u; bottom:Footprint (none) -> revxlp:empty; top:Footprint (none) -> revxlp:pg1350_plate_cut
- SwA1, SwA2, SwA3, SwA4, SwA5, SwAltG2, SwB1, SwB2, SwB3, SwB4, SwB5, SwC1, SwC2, SwC3, SwC4, SwC5, SwD1, SwD2, SwD3, SwD4, SwD5, SwE1, SwE2, SwE3, SwE4, SwE5, SwF1, SwF2, SwF3, SwF4, SwF5, SwG0, SwG1, SwG2, SwG3, SwG4, SwG5: symbol Switch:SW_Push_LED -> revxlp:SW_Push_LED; 10u-bottom:Footprint (none) -> revxlp:empty; 10u-top:Footprint (none) -> revxlp:pg1350_plate_cut; 10u:Footprint (none) -> revxlp:PG1350_socket_smdLed; Config (none) -> +top, +10u; bottom:Footprint (none) -> revxlp:empty; top:Footprint (none) -> revxlp:pg1350_plate_cut
- U1: symbol 74xx:74HC595 -> revxlp:74HC595; 10u-bottom:Footprint (none) -> revxlp:empty; 10u-top:Footprint (none) -> revxlp:empty; 10u:Footprint (none) -> Package_SO:SOIC-16_3.9x9.9mm_P1.27mm; Config (none) -> +10u; bottom:Footprint (none) -> revxlp:empty; top:Footprint (none) -> revxlp:empty
- U2: symbol Seeeduino XIAO:SeeeduinoXIAO_BLE -> revxlp:SeeeduinoXIAO_BLE; 10u-bottom:Footprint (none) -> revxlp:empty; 10u-top:Footprint (none) -> revxlp:empty; 10u:Footprint (none) -> zaphod:Seeeduino XIAO-MOUDLE14P-2.54-21X17.8MM; Config (none) -> +10u; bottom:Footprint (none) -> revxlp:empty; top:Footprint (none) -> revxlp:empty

Commit message: update .gitignore
Parts:
- BT1: 10u:Footprint revxlp:cell_pads -> (none)
Changed lines of the file:
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@@
 			)
 		)
-		(property "10u:Footprint" "revxlp:cell_pads"
+		(property "10u:Footprint" ""
 			(at 269.24 149.86 0)
 			(effects
